Commit message: feat(planner): Update planner parameters and TF frame references
- Changed the reference frame for the robot state from `base_link` to `rear_axle_link` in planner_params.yaml and planner_node.cpp.
- Adjusted the rear axle offset to match the URDF configuration.
- Updated the goal pose handling to account for the new reference frame.
- Modified the planner's TF lookup methods to use the new robot state frame.
- Enhanced the goal planning logic to shift the target based on the rear axle position.
- Updated the robot configuration files to reflect changes in TF frames and parameters.
- Improved command rate limiting in the NeupanCore class to ensure smoother control commands.
- Added new parameters for obstacle avoidance and refined existing ones in planner.yaml.
- Enhanced logging for better debugging and monitoring of the planning process.

File: src/ackermann_robot/xacro/chassis.xacro (robot description, xacro)
@@ -29,4 +29,15 @@
         </collision>
     </link>
+    <!--
+        NeuPAN and Hybrid A* use the rear axle center as the Ackermann
+        bicycle-model reference point.  Keep base_link as the vehicle/odom
+        reference used by ros2_control and robot_localization.
+    -->
+    <link name="rear_axle_link"/>
+    <joint name="rear_axle_joint" type="fixed">
+        <origin xyz="-0.30449 0 0.045" rpy="0 0 0" />
+        <parent link="base_link" />
+        <child link="rear_axle_link" />
+    </joint>
     <!-- <joint name="base_joint" type="fixed">
         <parent link="base_footprint"/>
