Commit message: 项目重构

File: src/ackermann_description/xacro/chassis.xacro (robot description, xacro)
@@ -18,5 +18,5 @@
             <origin xyz="0 0 0" rpy="0 0 0" />
             <geometry>
-                <mesh filename="package://ackermann_robot/meshes/top_akm_bs_robot_meshes/base_link.STL" />
+                <mesh filename="package://ackermann_description/meshes/top_akm_bs_robot_meshes/base_link.STL" />
             </geometry>
             <material name="blue"/>
@@ -60,5 +60,5 @@
                 <origin xyz="0 0 0" rpy="0 0 0" />
                 <geometry>
-                    <mesh filename="package://ackermann_robot/meshes/top_akm_bs_robot_meshes/${prefix}_rear_wheel_link.STL" />
+                    <mesh filename="package://ackermann_description/meshes/top_akm_bs_robot_meshes/${prefix}_rear_wheel_link.STL" />
                 </geometry>
                 <material name="white"/>
@@ -100,5 +100,5 @@
             <visual>
                 <geometry>
-                    <mesh filename="package://ackermann_robot/meshes/top_akm_bs_robot_meshes/${prefix}_steering_link.STL" />
+                    <mesh filename="package://ackermann_description/meshes/top_akm_bs_robot_meshes/${prefix}_steering_link.STL" />
                 </geometry>
                 <material name="blue"/>
@@ -106,5 +106,5 @@
             <collision>
                 <geometry>
-                    <mesh filename="package://ackermann_robot/meshes/top_akm_bs_robot_meshes/${prefix}_steering_link.STL" />
+                    <mesh filename="package://ackermann_description/meshes/top_akm_bs_robot_meshes/${prefix}_steering_link.STL" />
                 </geometry>
             </collision>
@@ -126,5 +126,5 @@
             <visual>
                 <geometry>
-                    <mesh filename="package://ackermann_robot/meshes/top_akm_bs_robot_meshes/${prefix}_front_wheel_link.STL" />
+                    <mesh filename="package://ackermann_description/meshes/top_akm_bs_robot_meshes/${prefix}_front_wheel_link.STL" />
                 </geometry>
                 <material name="white"/>

File: src/ackermann_description/xacro/control.xacro (robot description, xacro)
@@ -48,5 +48,5 @@
     <gazebo>
         <plugin filename="libgazebo_ros2_control.so" name="gazebo_ros2_control">
-            <parameters>$(find ackermann_robot)/config/ackermann_controllers.yaml</parameters>
+            <parameters>$(find ackermann_control)/config/ackermann_controllers.yaml</parameters>
             <ros>
                 <remapping>/ackermann_steering_controller/odometry:=/odom_wheel</remapping>

File: src/ackermann_description/xacro/sensors.xacro (robot description, xacro)
@@ -8,5 +8,5 @@
         </inertial>
         <visual>
-            <geometry> <mesh filename="package://ackermann_robot/meshes/top_akm_bs_robot_meshes/laser_link.STL" /> </geometry>
+            <geometry> <mesh filename="package://ackermann_description/meshes/top_akm_bs_robot_meshes/laser_link.STL" /> </geometry>
             <material name="white"/>
         </visual>
@@ -77,9 +77,9 @@
         </inertial>
         <visual>
-            <geometry> <mesh filename="package://ackermann_robot/meshes/top_akm_bs_robot_meshes/flaser.STL" /> </geometry>
+            <geometry> <mesh filename="package://ackermann_description/meshes/top_akm_bs_robot_meshes/flaser.STL" /> </geometry>
             <material name="grey"/>
         </visual>
         <collision>
-            <geometry> <mesh filename="package://ackermann_robot/meshes/top_akm_bs_robot_meshes/flaser.STL" /> </geometry>
+            <geometry> <mesh filename="package://ackermann_description/meshes/top_akm_bs_robot_meshes/flaser.STL" /> </geometry>
         </collision>
     </link>
@@ -118,9 +118,9 @@
         </inertial>
         <visual>
-            <geometry> <mesh filename="package://ackermann_robot/meshes/top_akm_bs_robot_meshes/camera_link.STL" /> </geometry>
+            <geometry> <mesh filename="package://ackermann_description/meshes/top_akm_bs_robot_meshes/camera_link.STL" /> </geometry>
             <material name="white"/>
         </visual>
         <collision>
-            <geometry> <mesh filename="package://ackermann_robot/meshes/top_akm_bs_robot_meshes/camera_link.STL" /> </geometry>
+            <geometry> <mesh filename="package://ackermann_description/meshes/top_akm_bs_robot_meshes/camera_link.STL" /> </geometry>
         </collision>
     </link>
@@ -177,9 +177,9 @@
         </inertial>
         <visual>
-            <geometry> <mesh filename="package://ackermann_robot/meshes/top_akm_bs_robot_meshes/gyro_link.STL" /> </geometry>
+            <geometry> <mesh filename="package://ackermann_description/meshes/top_akm_bs_robot_meshes/gyro_link.STL" /> </geometry>
             <material name="blue"/>
         </visual>
         <collision>
-            <geometry> <mesh filename="package://ackermann_robot/meshes/top_akm_bs_robot_meshes/gyro_link.STL" /> </geometry>
+            <geometry> <mesh filename="package://ackermann_description/meshes/top_akm_bs_robot_meshes/gyro_link.STL" /> </geometry>
         </collision>
     </link>
@@ -219,9 +219,9 @@
         </inertial>
         <visual>
-            <geometry> <mesh filename="package://ackermann_robot/meshes/top_akm_bs_robot_meshes/rtk_link.STL" /> </geometry>
+            <geometry> <mesh filename="package://ackermann_description/meshes/top_akm_bs_robot_meshes/rtk_link.STL" /> </geometry>
             <material name="white"/>
         </visual>
         <collision>
-             <geometry> <mesh filename="package://ackermann_robot/meshes/top_akm_bs_robot_meshes/rtk_link.STL" /> </geometry>
+             <geometry> <mesh filename="package://ackermann_description/meshes/top_akm_bs_robot_meshes/rtk_link.STL" /> </geometry>
         </collision>
     </link>
