Commit message: feat: native hybrid A* planner + NeuPAN tuning + docs
Major changes:
- Integrate standalone hybrid_astar_planner (OMPL SE2 A*) replacing Nav2 SmacPlannerHybrid
- PGMMapAdapter: direct PGM binary read with Y-axis flip, Nav2 cost convention
- planner_node: TF-based map->base_link lookup (hdl_localization), /plan topic for NeuPAN
- navigation_hdl.launch.py: hybrid-a-star + hdl + pcl_to_scan + cmd_vel_mux (no Nav2)
- Docs: NeuPAN MPC tuning guide with robot-scale normalization (docs/neupan_tuning.md)
- NeuPAN planner.yaml: tuned q_s/p_u/eta for 0.7m robot (L0=0.7m, v0=1.0m/s)

Submodule restructure:
- hdl_localization: moved under src/hdl_localization/src/ with fast_gicp, hdl_global_localization, ndt_omp
- Removed old top-level ndt_omp and hdl_localization flat files

Config updates:
- RViz: nav2 GoalTool -> rviz_default_plugins/SetGoal (/goal_pose)
- Robot URDF, EKF config, LIO-SAM params, Gazebo launch
- Nav2 params cleared (no longer used)

Scripts: nav_hdl_neupan.sh, run_neupan.sh

File: src/LIO-SAM/config/robot.urdf.xacro (robot description, xacro)
@@ -2,33 +2,16 @@
 <robot name="lio" xmlns:xacro="http://tixiaoshan.github.io/">
   <xacro:property name="PI" value="3.1415926535897931" />
-  <link name="chassis_link"></link>
+  <!-- AckermannRobot-3D frame structure for LIO-SAM visualization -->
   <link name="base_link"></link>
-  <joint name="base_link_joint" type="fixed">
-    <parent link="base_link"/>
-    <child link="chassis_link" />
-    <origin xyz="0 0 0" rpy="0 0 0" />
+  <link name="laser_link"> </link>
+  <joint name="laser_joint" type="fixed">
+    <parent link="base_link" />
+    <child link="laser_link" />
+    <origin xyz="-0.078 0.0 0.384" rpy="0 0 0" />
   </joint>
-  <link name="lidar_link"> </link>
-  <joint name="lidar_joint" type="fixed">
+  <link name="gyro_link"> </link>
+  <joint name="gyro_joint" type="fixed">
     <parent link="base_link" />
-    <child link="lidar_link" />
-    <origin xyz="0 0 0" rpy="0 0 0" />
-  </joint>
-  <link name="imu_link"> </link>
-  <joint name="imu_joint" type="fixed">
-    <parent link="chassis_link" />
-    <child link="imu_link" />
-    <origin xyz="0 0 0" rpy="0 0 0" />
-  </joint>
-  <link name="laser_sensor_frame"> </link>
-  <joint name="laser_joint" type="fixed">
-    <parent link="imu_link" />
-    <child link="laser_sensor_frame" />
-    <origin xyz="0 0 0" rpy="0 0 0" />
-  </joint>
-  <link name="navsat_link"> </link>
-  <joint name="navsat_joint" type="fixed">
-    <parent link="chassis_link" />
-    <child link="navsat_link" />
+    <child link="gyro_link" />
     <origin xyz="0 0 0" rpy="0 0 0" />
   </joint>

Commit message: feat: Integrate IMU pose and LIO-SAM extrinsics into vehicle configuration
- Added functions `imu_transform()` and `lio_sam_extrinsics()` to compute static transforms and extrinsic parameters from the vehicle configuration.
- Updated tests to validate IMU and LiDAR transforms, ensuring consistency with the new configuration.
- Introduced a new CSV recording script for Allan variance analysis of IMU data.
- Created a launch file for LIO-SAM mapping, consolidating sensor data sources and static transforms.
- Enhanced IMU calibration scripts for better noise parameter extraction.
- Documented the integration process and configuration changes in `imu_lio_sam_integration.md`.

File: src/LIO-SAM/config/robot.urdf.xacro (robot description, xacro)
@@ -8,11 +8,15 @@
     <parent link="base_link" />
     <child link="laser_link" />
-    <origin xyz="-0.078 0.0 0.384" rpy="0 0 0" />
+    <origin xyz="0.99 0.0 0.66" rpy="0 0 0" />
   </joint>
+  <!-- 注意：gyro_joint 的值是 vehicle_config 的手工同步拷贝，仅供本 xacro 可视化。
+       当前未被任何 launch 的 robot_state_publisher 消费；唯一数据源为
+       src/vehicle_config/config/real_vehicle.yaml 的 sensors.imu.mount。
+       LIO-SAM 实际使用的外参由 run.launch.py 注入，与本 xacro 无关。 -->
   <link name="gyro_link"> </link>
   <joint name="gyro_joint" type="fixed">
     <parent link="base_link" />
     <child link="gyro_link" />
-    <origin xyz="0 0 0" rpy="0 0 0" />
+    <origin xyz="0.13 0.0 0.26" rpy="-0.006945 -0.006617 0.0" />
   </joint>
 </robot>
