Commit message: 按功能分层整理ROS包并重命名

File: src/simulation/robot/xacro/chassis.xacro (robot description, xacro)
@@ -18,5 +18,5 @@
             <origin xyz="0 0 0" rpy="0 0 0" />
             <geometry>
-                <mesh filename="package://ackermann_simulation/robot/meshes/top_akm_bs_robot_meshes/base_link.STL" />
+                <mesh filename="package://simulation/robot/meshes/top_akm_bs_robot_meshes/base_link.STL" />
             </geometry>
             <material name="blue"/>
@@ -60,5 +60,5 @@
                 <origin xyz="0 0 0" rpy="0 0 0" />
                 <geometry>
-                    <mesh filename="package://ackermann_simulation/robot/meshes/top_akm_bs_robot_meshes/${prefix}_rear_wheel_link.STL" />
+                    <mesh filename="package://simulation/robot/meshes/top_akm_bs_robot_meshes/${prefix}_rear_wheel_link.STL" />
                 </geometry>
                 <material name="white"/>
@@ -100,5 +100,5 @@
             <visual>
                 <geometry>
-                    <mesh filename="package://ackermann_simulation/robot/meshes/top_akm_bs_robot_meshes/${prefix}_steering_link.STL" />
+                    <mesh filename="package://simulation/robot/meshes/top_akm_bs_robot_meshes/${prefix}_steering_link.STL" />
                 </geometry>
                 <material name="blue"/>
@@ -106,5 +106,5 @@
             <collision>
                 <geometry>
-                    <mesh filename="package://ackermann_simulation/robot/meshes/top_akm_bs_robot_meshes/${prefix}_steering_link.STL" />
+                    <mesh filename="package://simulation/robot/meshes/top_akm_bs_robot_meshes/${prefix}_steering_link.STL" />
                 </geometry>
             </collision>
@@ -126,5 +126,5 @@
             <visual>
                 <geometry>
-                    <mesh filename="package://ackermann_simulation/robot/meshes/top_akm_bs_robot_meshes/${prefix}_front_wheel_link.STL" />
+                    <mesh filename="package://simulation/robot/meshes/top_akm_bs_robot_meshes/${prefix}_front_wheel_link.STL" />
                 </geometry>
                 <material name="white"/>

File: src/simulation/robot/xacro/sensors.xacro (robot description, xacro)
@@ -8,5 +8,5 @@
         </inertial>
         <visual>
-            <geometry> <mesh filename="package://ackermann_simulation/robot/meshes/top_akm_bs_robot_meshes/laser_link.STL" /> </geometry>
+            <geometry> <mesh filename="package://simulation/robot/meshes/top_akm_bs_robot_meshes/laser_link.STL" /> </geometry>
             <material name="white"/>
         </visual>
@@ -77,9 +77,9 @@
         </inertial>
         <visual>
-            <geometry> <mesh filename="package://ackermann_simulation/robot/meshes/top_akm_bs_robot_meshes/flaser.STL" /> </geometry>
+            <geometry> <mesh filename="package://simulation/robot/meshes/top_akm_bs_robot_meshes/flaser.STL" /> </geometry>
             <material name="grey"/>
         </visual>
         <collision>
-            <geometry> <mesh filename="package://ackermann_simulation/robot/meshes/top_akm_bs_robot_meshes/flaser.STL" /> </geometry>
+            <geometry> <mesh filename="package://simulation/robot/meshes/top_akm_bs_robot_meshes/flaser.STL" /> </geometry>
         </collision>
     </link>
@@ -118,9 +118,9 @@
         </inertial>
         <visual>
-            <geometry> <mesh filename="package://ackermann_simulation/robot/meshes/top_akm_bs_robot_meshes/camera_link.STL" /> </geometry>
+            <geometry> <mesh filename="package://simulation/robot/meshes/top_akm_bs_robot_meshes/camera_link.STL" /> </geometry>
             <material name="white"/>
         </visual>
         <collision>
-            <geometry> <mesh filename="package://ackermann_simulation/robot/meshes/top_akm_bs_robot_meshes/camera_link.STL" /> </geometry>
+            <geometry> <mesh filename="package://simulation/robot/meshes/top_akm_bs_robot_meshes/camera_link.STL" /> </geometry>
         </collision>
     </link>
@@ -177,9 +177,9 @@
         </inertial>
         <visual>
-            <geometry> <mesh filename="package://ackermann_simulation/robot/meshes/top_akm_bs_robot_meshes/gyro_link.STL" /> </geometry>
+            <geometry> <mesh filename="package://simulation/robot/meshes/top_akm_bs_robot_meshes/gyro_link.STL" /> </geometry>
             <material name="blue"/>
         </visual>
         <collision>
-            <geometry> <mesh filename="package://ackermann_simulation/robot/meshes/top_akm_bs_robot_meshes/gyro_link.STL" /> </geometry>
+            <geometry> <mesh filename="package://simulation/robot/meshes/top_akm_bs_robot_meshes/gyro_link.STL" /> </geometry>
         </collision>
     </link>
@@ -219,9 +219,9 @@
         </inertial>
         <visual>
-            <geometry> <mesh filename="package://ackermann_simulation/robot/meshes/top_akm_bs_robot_meshes/rtk_link.STL" /> </geometry>
+            <geometry> <mesh filename="package://simulation/robot/meshes/top_akm_bs_robot_meshes/rtk_link.STL" /> </geometry>
             <material name="white"/>
         </visual>
         <collision>
-             <geometry> <mesh filename="package://ackermann_simulation/robot/meshes/top_akm_bs_robot_meshes/rtk_link.STL" /> </geometry>
+             <geometry> <mesh filename="package://simulation/robot/meshes/top_akm_bs_robot_meshes/rtk_link.STL" /> </geometry>
         </collision>
     </link>
